Commit message: elfin5

File: elfin5/elfin5_ros2_gazebo/urdf/elfin5.urdf.xacro (robot description, xacro)
@@ -1,6 +1,5 @@
 <?xml version="1.0"?>
 <robot name="elfin5" xmlns:xacro="http://wiki.ros.org/xacro">
-  <xacro:arg name="use_real_hardware" default="true" />
-  <xacro:arg name="use_fake_hardware" default="false" />
+  <xacro:macro name="elfin5_ros2_gazebo_urdf" params="use_real_hardware use_fake_hardware">
   <!-- Load TRANSMISSION file: -->
   <xacro:include filename="$(find elfin5_ros2_gazebo)/urdf/elfin5_transmission.xacro" />
@@ -13,6 +12,6 @@
     <!-- GAZEBO - ROS2_CONTROL: -->
     <xacro:elfin5_gazebo
-    use_real_hardware="$(arg use_real_hardware)"
-    use_fake_hardware="$(arg use_fake_hardware)"/>
+    use_real_hardware="${use_real_hardware}"
+    use_fake_hardware="${use_fake_hardware}"/>
   <link name="world"/>
   <joint name="world_base" type="fixed">
@@ -448,3 +447,4 @@
       link="elfin_dummy_gripper" />
   </joint>
+  </xacro:macro>
 </robot>
