Commit message: elfin10

File: elfin10/elfin10_ros2_gazebo/urdf/elfin10.urdf.xacro (robot description, xacro)
@@ -1,6 +1,5 @@
 <?xml version="1.0"?>
 <robot name="elfin10" xmlns:xacro="http://wiki.ros.org/xacro">
-  <xacro:arg name="use_real_hardware" default="true" />
-  <xacro:arg name="use_fake_hardware" default="false" />
+  <xacro:macro name="elfin10_ros2_gazebo_urdf" params="use_real_hardware use_fake_hardware">
   <!-- Load TRANSMISSION file: -->
   <xacro:include filename="$(find elfin10_ros2_gazebo)/urdf/elfin10_transmission.xacro" />
@@ -14,11 +13,13 @@
     <!-- GAZEBO - ROS2_CONTROL: -->
     <xacro:elfin10_gazebo
-    use_real_hardware="$(arg use_real_hardware)"
-    use_fake_hardware="$(arg use_fake_hardware)"/>
+    use_real_hardware="${use_real_hardware}"
+    use_fake_hardware="${use_fake_hardware}"/>
    <link name="world"/>
+  <!-- NOTE: 不知道为啥这个默认绕z转了-90度
+         之前是 rpy="0 0 -1.5708" -->
   <joint name="world_base" type="fixed">
     <origin
       xyz="0 0 0"
-      rpy="0 0 -1.5708" />
+      rpy="0 0 0" />
     <parent
       link="world" />
@@ -449,3 +450,4 @@
       link="elfin_dummy_gripper" />
   </joint>
+  </xacro:macro>
 </robot>

File: elfin10/elfin10_ros2_gazebo/urdf/elfin10_gazebo.xacro (robot description, xacro)
@@ -14,8 +14,11 @@
         <xacro:if value="${use_real_hardware}">
           <plugin>elfin_hardware_interface/ElfinHWInterface</plugin>
+          <param name="main_loop_update_rate">250.0</param>
+          <param name="desired_hw_update_rate">250.0</param>
         </xacro:if>
         <xacro:unless value="${use_real_hardware}">
           <xacro:if value="${use_fake_hardware}">
-              <plugin>fake_components/GenericSystem</plugin>
+              <plugin>mock_components/GenericSystem</plugin>
+              <param name="state_following_offset">0.0</param>
           </xacro:if>
           <xacro:unless value="${use_fake_hardware}">
